File: hardware/Breakout_104pin_EEC-V-Connector/eecv-breakout.kicad_pcb (KiCad board)
At the start: 4 copper layers, 140.8 x 53.7 mm, 12 parts, among them J1 EEC-V, J2 Conn_01x13, J3 Conn_01x13, J4 Conn_01x13, J5 Conn_01x13, J6 Conn_01x13, J7 Conn_01x13, J8 Conn_01x13, J9 Conn_01x13

Commit message: test bump
Other:
- board text added: "rusefi.com Rev. 0.3 foo"
- board text removed: "rusefi.com Rev. 0.3"

Commit message: test poke
Other:
- board text added: "rusefi.com Rev. 0.3 foobar"
- board text removed: "rusefi.com Rev. 0.3 foo"
Changed lines of the file:
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@@
     (effects (font (size 1 1) (thickness 0.15)))
   )
-  (gr_text "rusefi.com    Rev. 0.3 foo" (at 159.406 54.352 270) (layer "F.SilkS")
+  (gr_text "rusefi.com    Rev. 0.3 foobar" (at 159.406 54.352 270) (layer "F.SilkS")
     (effects (font (size 1 1) (thickness 0.15)))
   )
