File: hardware/Breakout_112pin_Connector/Breakout_112pin_Connector.kicad_pcb (KiCad board)
At the start: 2 copper layers, 174 x 58 mm, 42 parts, among them J1 0643330100, J10 Conn_01x06, J11 Conn_01x06, J12 Conn_01x06, J13 Conn_01x06, J14 Conn_01x04, J15 Conn_01x04, J16 Conn_01x06, J17 Conn_01x06, J18 Conn_01x06, J19 Conn_01x06, J2 Conn_01x04, J20 Conn_01x04, J21 Conn_01x04, J22 Conn_01x06, J23 Conn_01x06, J24 Conn_01x06, J25 Conn_01x06, J26 Conn_01x01, J27 Conn_01x01, J28 Conn_01x04, J29 Conn_01x04, J3 Conn_01x04, J30 Conn_01x10, J31 Conn_01x10, J32 Conn_01x10, J33 Conn_01x10, J34 Conn_01x04, J35 Conn_01x04, J36 Conn_01x10, J37 Conn_01x10, J38 Conn_01x10, J39 Conn_01x10, J4 Conn_01x06, J5 Conn_01x06, J6 Conn_01x06, J7 Conn_01x06, J8 Conn_01x04, J9 Conn_01x04

Commit message: update pcb files
Other:
- net class Default removed
