File: hardware/Breakout_121pin_368255-2-Connector/368255-2.kicad_pcb (KiCad board)
At the start: 2 copper layers, 146.1 x 49.5 mm, 43 parts, among them P1 368255-2, P10 CONN_1, P11 CONN_1, P12 CONN_1, P13 CONN_1, P14 CONN_1, P15 CONN_1, P16 CONN_1, P17 CONN_1, P18 CONN_1, P19 CONN_1, P2 CONN_19, P20 CONN_1, P21 CONN_1, P22 CONN_1, P23 CONN_1, P24 CONN_1, P25 CONN_1, P26 CONN_1, P27 CONN_1, P28 CONN_1, P29 CONN_1, P3 CONN_19, P30 CONN_1, P31 CONN_1, P32 CONN_8, P33 CONN_8, P34 CONN_8, P35 CONN_8, P36 CONN_1, P37 CONN_1, P4 CONN_19, P5 CONN_19, P6 CONN_1, P7 CONN_1, P8 CONN_1, P9 CONN_1

Commit message: update pcb files
Other:
- net class 1.5A removed
- net class 10A removed
- net class 1A removed
- net class 3.75A removed
- net class Default removed
