File: hardware/Breakout_134pin_7-967288-1-Connector/134pin_7-967288-1.kicad_pcb (KiCad board)
At the start: 2 copper layers, 139.7 x 73.7 mm, 40 parts, among them J1 Conn_01x03, J10 Conn_01x06, J11 Conn_01x06, J12 Conn_01x03, J13 Conn_01x03, J14 Conn_01x03, J15 Conn_01x13, J16 Conn_01x13, J17 Conn_01x13, J18 Conn_01x13, J19 Conn_01x13, J2 Conn_01x03, J20 Conn_01x13, J21 Conn_01x13, J22 Conn_01x13, J23 Conn_01x10, J24 Conn_01x10, J25 Conn_01x10, J26 Conn_01x10, J27 Conn_01x03, J28 Conn_01x03, J29 Conn_01x03, J3 Conn_01x03, J30 Conn_01x10, J31 Conn_01x10, J32 Conn_01x10, J33 Conn_01x10, J34 Conn_01x03, J35 Conn_01x03, J36 Conn_01x03, J37 Conn_01x01, J4 Conn_01x06, J5 Conn_01x06, J6 Conn_01x06, J7 Conn_01x06, J8 Conn_01x06, J9 Conn_01x06, P1 134pin_7-967288-1_KC5

Commit message: update pcb files
Other:
- net class 1A EXTERNAL removed
- net class 2.5A EXTERNAL removed
- net class 3,5A EXT HIGH VOLTAGE removed
- net class 3.5A EXTERNAL removed
- net class 5A EXTERNAL removed
- net class CUSTOM removed
- net class CUSTOM 0.6 removed
- net class Default removed
- net class MIN_EXTERN_188A removed
- net class MIN_EXTERN_241A removed
