File: hardware/Breakout_38pin_NGC-connector/NGC_38_connector.kicad_pcb (KiCad board)
At the start: 2 copper layers, 31.8 x 47.6 mm, 9 parts, among them P1 DIL38, P2 CONN_10, P3 CONN_9, P4 CONN_10, P5 CONN_9, P6 CONN_10, P7 CONN_9, P8 CONN_9, P9 CONN_10

Commit message: update pcb files
Other:
- net class Default removed
