File: hardware/Breakout_48pin_174917-Connector/174917.kicad_pcb (KiCad board)
At the start: 2 copper layers, 100 x 33.5 mm, 39 parts, among them P1 CONN_3, P10 CONN_1, P11 CONN_1, P12 CONN_1, P13 CONN_3, P14 CONN_3, P15 CONN_1, P16 CONN_1, P17 CONN_1, P18 CONN_1, P19 CONN_1, P2 CONN_3, P20 CONN_1, P21 CONN_1, P22 CONN_1, P23 CONN_1, P24 CONN_1, P25 174917, P26 CONN_8, P27 CONN_8, P3 CONN_1, P30 CONN_8, P31 CONN_8, P32 CONN_8, P33 CONN_8, P36 CONN_8, P37 CONN_8, P38 CONN_1, P39 CONN_1, P4 CONN_1, P40 CONN_1, P41 CONN_1, P5 CONN_1, P6 CONN_1, P7 CONN_1, P8 CONN_1, P9 CONN_1

Commit message: update pcb files
Routing:
- net Net-(P25-Pad25): track 20.3 -> 0.00 mm
- net Net-(P25-Pad2C): track 0.00 -> 20.3 mm
- net Net-(P25-Pad44): track 18.8 -> 0.00 mm
- net Net-(P25-Pad2V): track 0.00 -> 18.8 mm
- net Net-(P25-Pad2D): track 0.00 -> 18.8 mm
- net Net-(P25-Pad26): track 18.8 -> 0.00 mm
- net Net-(P25-Pad43): track 18.8 -> 0.00 mm
- net Net-(P25-Pad2U): track 0.00 -> 18.8 mm
- net Net-(P25-Pad27): track 18.7 -> 0.00 mm
- net Net-(P25-Pad2E): track 0.00 -> 18.7 mm
- net Net-(P25-Pad45): track 18.6 -> 0.00 mm
- net Net-(P25-Pad2W): track 0.00 -> 18.6 mm
- net Net-(P25-Pad31): track 18.4 -> 0.00 mm
- net Net-(P25-Pad2I): track 0.00 -> 18.4 mm
- net Net-(P25-Pad46): track 18.4 -> 0.00 mm
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Other:
- net class 1.5A removed
- net class 10A removed
- net class 1A removed
- net class 3.75A removed
- net class Default removed
