File: hardware/Breakout_52pin_172319-1-Connector/172319-1_connector.kicad_pcb (KiCad board)
At the start: 2 copper layers, 124.5 x 33.7 mm, 3 parts, among them P1 172319-1, P2 172319-1, P3 CONN_01X01

Commit message: update pcb files
Other:
- net class 2.5A-1Oz_ext removed
- net class Default removed
