File: hardware/Breakout_55pin-motronic-Connector/motronic-wire-adapter.kicad_pcb (KiCad board)
At the start: 2 copper layers, 157.5 x 48.5 mm, 10 parts, among them P1 MOTRONIC, P2 CONN_19, P3 CONN_18, P4 CONN_18, P5 CONN_1, P6 CONN_1

Commit message: update pcb files
Other:
- net class Default removed
