File: hardware/Breakout_55pin_963063-15-Connector/963063-15.kicad_pcb (KiCad board)
At the start: 2 copper layers, 150 x 50 mm, 10 parts, among them P1 963063_15, P2 CONN_19, P3 CONN_18, P4 CONN_18, P5 CONN_1, P6 CONN_1

Commit message: update pcb files
Other:
- net class Default removed
