File: hardware/Breakout_64pin_176122-6-Connector/176122-6.kicad_pcb (KiCad board)
At the start: 2 copper layers, 137.2 x 41.5 mm, 28 parts, among them P1 CONN_3, P13 CONN_3, P14 CONN_3, P19 CONN_1, P2 CONN_3, P20 CONN_1, P25 0176122-06, P26 CONN_8, P27 CONN_8, P28 CONN_8, P29 CONN_8, P3 Conn_01x04_Male, P30 CONN_8, P31 CONN_8, P32 CONN_8, P33 CONN_8, P34 CONN_8, P35 CONN_8, P36 CONN_8, P37 CONN_8, P4 Conn_01x04_Male, P42 Conn_01x04_Male, P43 Conn_01x04_Male, P7 CONN_1, P8 CONN_1

Commit message: update pcb files
Other:
- net class Default removed
