File: hardware/Breakout_68pin_966595-1_and_963356-1-Connector/966595-1_and_963356-1.kicad_pcb (KiCad board)
At the start: 2 copper layers, 116 x 33 mm, 4 parts, among them P101 963356-1, P102 966595-1

Commit message: update pcb files
Other:
- net class 1.5A removed
- net class 10A removed
- net class 1A removed
- net class 3.75A removed
- net class Default removed
