File: hardware/Breakout_80pin_8-1393476-0/Breakout_80pin_1393476-Connector.kicad_pcb (KiCad board)
At the start: 2 copper layers, 144 x 58 mm, 24 parts, among them J1 8-1393476-0, J10 Conn_01x12, J11 Conn_01x14, J12 Conn_01x12, J13 Conn_01x14, J14 Conn_01x12, J15 Conn_01x12, J16 Conn_01x01, J17 Conn_01x01, J18 Conn_01x01, J19 Conn_01x01, J2 Conn_01x12, J20 Screw_Terminal_01x02, J21 Screw_Terminal_01x02, J3 Conn_01x12, J4 Conn_01x14, J5 Conn_01x12, J6 Screw_Terminal_01x02, J7 Conn_01x12, J8 Conn_01x14, J9 Screw_Terminal_01x02

Commit message: update pcb files
Other:
- net class Default removed
