File: hardware/Breakout_Chip_TLE6244/Breakout_TLE6244.kicad_pcb (KiCad board)
At the start: 4 copper layers, 50.8 x 38.1 mm, 73 parts, among them K1 CONN_3, K2 CONN_3, K3 CONN_3, K4 CONN_3, K5 CONN_3, K6 CONN_3, K7 CONN_3, P1 CONN_4, P2 CONN_3, P3 CONN_2, P4 CONN_3, P5 CONN_5, P6 CONN_3, P7 CONN_2, P8 CONN_2, U1 TLE6244

Commit message: update pcb files
Routing:
- added copper zone on In1.Cu, net /5v
- added copper zone on In2.Cu, net GND
- removed copper zone on PWR, net /5v
- removed copper zone on GND, net GND
Other:
- net class 1A external removed
- net class 2.5A external removed
- net class 3.5A external removed
- net class 5A external removed
- net class Default removed
- net class min2_extern_.188A removed
- net class min_extern_.241A removed
