File: hardware/CJ125_board/O2_input_CJ125.kicad_pcb (KiCad board)
At the start: 4 copper layers, 18.2 x 34.3 mm, 39 parts, among them P4 CONN_02X03, P8 CONN_02X05, Q1 FDS2734, U1 CJ125

Commit message: update pcb files
Routing:
- added copper zone on In1.Cu, net /CJ125_5v
- added copper zone on In1.Cu, net /WO2-12V
- added copper zone on In2.Cu, net GND
- removed copper zone on PWR, net /CJ125_5v
- removed copper zone on PWR, net /WO2-12V
- removed copper zone on GND, net GND
Other:
- net class 1A external removed
- net class 2.5A external removed
- net class 3.5A external removed
- net class 5A external removed
- net class Default removed
- net class min2_extern_.188A removed
- net class min_extern_.241A removed
