File: hardware/DDPAK_breakout/DDPAK_breakout.kicad_pcb (KiCad board)
At the start: 2 copper layers, 19.7 x 21.6 mm, 6 parts, among them P1 CONN_1, P2 CONN_2, P3 CONN_1, Q1 IRGS14C40L

Commit message: update pcb files
Other:
- net class Default removed
- net class FAT removed
- net class MIN removed
