File: hardware/EEC-V-Blank-Board/eecv.kicad_pcb (KiCad board)
At the start: 2 copper layers, 140.8 x 164.4 mm, 1 part, among them J1 EEC-V

Commit message: update pcb files
Other:
- net class Default removed
