File: hardware/Power_regulator_TPS54340/TPS54340_Buck_Regulator.kicad_pcb (KiCad board)
At the start: 2 copper layers, 26 x 15.9 mm, 20 parts, among them J1 Conn_01x01, J2 Conn_01x01, J3 Conn_01x01, J4 Conn_01x01, J5 Conn_01x01, U1 TPS54340

Commit message: update pcb files
Other:
- net class 1A_EXTERNAL removed
- net class 3.5A_EXTERNAL removed
- net class 5A_EXTERNAL removed
- net class Default removed
- net class PIN_WIDTH removed
