File: hardware/VR_discrete/vr_mmm.kicad_pcb (KiCad board)
At the start: 2 copper layers, 40.6 x 15.2 mm, 30 parts, among them P1 CONN_4, P2 CONN_4, U1 LM2903

Commit message: update pcb files
Other:
- net class Default removed
