File: hardware/VR_ncv1124_test_module/ncv1124.kicad_pcb (KiCad board)
At the start: 2 copper layers, 65 x 46 mm, 35 parts, among them J1 Screw_Terminal_01x02, J2 Screw_Terminal_01x02, J3 Screw_Terminal_01x02, J4 Screw_Terminal_01x02, J5 Screw_Terminal_01x02, J6 Screw_Terminal_01x02, J7 Conn_01x02_Male, J8 Conn_01x03_Male, Q1 2N7002, Q2 2N7002

Commit message: update pcb files
Other:
- net class Default removed
