File: hardware/brain_board_SD_Card_1/brain_board_SD_Card_1.kicad_pcb (KiCad board)
At the start: 2 copper layers, 14.6 x 33 mm, 6 parts, among them P352 MICRO-SDCARD-CONNECTOR-330006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, P5 CONN_01X03, P6 CONN_01X03

Commit message: update pcb files
Other:
- net class Default removed
