File: hardware/brain_board_STM32F407_SD_wing-it/brain_board_STM32F407_SD_wing-it.kicad_pcb (KiCad board)
At the start: 2 copper layers, 7.9 x 39.1 mm, 8 parts, among them P1 CONN_02X04, P11 CONN_01X01, P12 CONN_01X01, P2 CONN_02X03, P5 CONN_01X03, P6 CONN_01X03, P7 CONN_01X01, P8 CONN_01X01

Commit message: update pcb files
Other:
- net class Default removed
