File: hardware/soic8_breakout/soic8_breakout.kicad_pcb (KiCad board)
At the start: 2 copper layers, 3 parts, among them P1 CONN_4, P2 CONN_4, U1 XTR116U

Commit message: update pcb files
Other:
- net class Default removed
